Commit message: simulated and joined Link3, Link4, Link5, Link6

File: body.urdf (robot description, URDF)
Before this commit: robot robot, 2 links, 1 joints
Links:
- added link Link2, mass 1; collision box size=1 1 1; visual box size=1 1 1
- added link Link3, mass 1; collision box size=1 1 1; visual box size=1 1 1
- added link Link4, mass 1; collision box size=1 1 1; visual box size=1 1 1
- added link Link5, mass 1; collision box size=1 1 1; visual box size=1 1 1
- added link Link6, mass 1; collision box size=1 1 1; visual box size=1 1 1
Joints:
- added joint Link1_Link2: type revolute, parent Link1, child Link2, origin xyz=0 0 1.0 rpy=0 0 0, axis 0 1 0, limit lower=-3.14159 upper=3.14159 effort=0.0 velocity=0.0
- added joint Link2_Link3: type revolute, parent Link2, child Link3, origin xyz=0 0.5 0.5 rpy=0 0 0, axis 0 1 0, limit lower=-3.14159 upper=3.14159 effort=0.0 velocity=0.0
- added joint Link3_Link4: type revolute, parent Link3, child Link4, origin xyz=0 1 0 rpy=0 0 0, axis 0 1 0, limit lower=-3.14159 upper=3.14159 effort=0.0 velocity=0.0
- added joint Link4_Link5: type revolute, parent Link4, child Link5, origin xyz=0 0.5 -0.5 rpy=0 0 0, axis 0 1 0, limit lower=-3.14159 upper=3.14159 effort=0.0 velocity=0.0
- added joint Link5_Link6: type revolute, parent Link5, child Link6, origin xyz=0 0 -1.5 rpy=0 0 0, axis 0 1 0, limit lower=-3.14159 upper=3.14159 effort=0.0 velocity=0.0

Commit message: legs in the air

File: body.urdf (robot description, URDF)
Before this commit: robot robot, 9 links, 8 joints
Links:
- removed link BackLowerLeg
- removed link FrontLowerLeg
- removed link LeftLowerLeg
- removed link RightLowerLeg
- added link BackLeft, mass 1; collision box size=0.2 0.2 1; visual box size=0.2 0.2 1
- added link BackRight, mass 1; collision box size=0.2 0.2 1; visual box size=0.2 0.2 1
- added link FrontLeft, mass 1; collision box size=0.2 0.2 1; visual box size=0.2 0.2 1
- added link FrontRight, mass 1; collision box size=0.2 0.2 1; visual box size=0.2 0.2 1
Joints:
- removed joint BackLeg_BackLowerLeg
- removed joint FrontLeg_FrontLowerLeg
- removed joint LeftLeg_LeftLowerLeg
- removed joint RightLeg_RightLowerLeg
- added joint Torso_BackLeft: type revolute, parent Torso, child BackLeft, origin xyz=-0.5 -0.5 1 rpy=0 0 0, axis 1 0 0, limit lower=-3.14159 upper=3.14159 effort=0.0 velocity=0.0
- added joint Torso_BackRight: type revolute, parent Torso, child BackRight, origin xyz=0.5 -0.5 1 rpy=0 0 0, axis 1 0 0, limit lower=-3.14159 upper=3.14159 effort=0.0 velocity=0.0
- added joint Torso_FrontLeft: type revolute, parent Torso, child FrontLeft, origin xyz=-0.5 0.5 1 rpy=0 0 0, axis 1 0 0, limit lower=-3.14159 upper=3.14159 effort=0.0 velocity=0.0
- added joint Torso_FrontRight: type revolute, parent Torso, child FrontRight, origin xyz=0.5 0.5 1 rpy=0 0 0, axis 1 0 0, limit lower=-3.14159 upper=3.14159 effort=0.0 velocity=0.0

Commit message: housekeeping, single link

File: body.urdf (robot description, URDF)
Before this commit: robot robot, 9 links, 8 joints
Links:
- removed link BackLeft
- removed link BackLeg
- removed link BackRight
- removed link FrontLeft
- removed link FrontLeg
- removed link FrontRight
- removed link LeftLeg
- removed link RightLeg
- removed link Torso
- added link base, mass 1; collision box size=0.33168802015290966 0.051877593284682666 0.6175933200728823; visual box size=0.33168802015290966 0.051877593284682666 0.6175933200728823
Joints:
- removed joint Torso_BackLeft
- removed joint Torso_BackLeg
- removed joint Torso_BackRight
- removed joint Torso_FrontLeft
- removed joint Torso_FrontLeg
- removed joint Torso_FrontRight
- removed joint Torso_LeftLeg
- removed joint Torso_RightLeg

Commit message: done.

File: body.urdf (robot description, URDF)
Before this commit: robot robot, 1 links, 0 joints
Links:
- removed link base
- added link Link0, mass 1; collision box size=0.5471109201794214 0.494838829967435 0.18890324347836876; visual box size=0.5471109201794214 0.494838829967435 0.18890324347836876
- added link Link1, mass 1; collision box size=1.0966786066332916 0.9067129132754954 1.1863614334945194; visual box size=1.0966786066332916 0.9067129132754954 1.1863614334945194
- added link Link2, mass 1; collision box size=0.5099032540277433 0.4060790194638573 1.19729578547389; visual box size=0.5099032540277433 0.4060790194638573 1.19729578547389
- added link Link3, mass 1; collision box size=0.7047107183574421 1.0521541731407715 0.677277913405836; visual box size=0.7047107183574421 1.0521541731407715 0.677277913405836
- added link Link4, mass 1; collision box size=0.33827715943261455 0.8361161104843533 0.9531082949139518; visual box size=0.33827715943261455 0.8361161104843533 0.9531082949139518
- added link Link5, mass 1; collision box size=1.061440823953466 1.0941545152718655 0.810925211551816; visual box size=1.061440823953466 1.0941545152718655 0.810925211551816
Joints:
- added joint Link0_Link1: type revolute, parent Link0, child Link1, origin xyz=0 0.2474194149837175 0.3 rpy=0 0 0, axis 1 0 0, limit lower=-3.14159 upper=3.14159 effort=0.0 velocity=0.0
- added joint Link1_Link2: type revolute, parent Link1, child Link2, origin xyz=0 0.9067129132754954 0 rpy=0 0 0, axis 1 0 0, limit lower=-3.14159 upper=3.14159 effort=0.0 velocity=0.0
- added joint Link2_Link3: type revolute, parent Link2, child Link3, origin xyz=0 0.4060790194638573 0 rpy=0 0 0, axis 1 0 0, limit lower=-3.14159 upper=3.14159 effort=0.0 velocity=0.0
- added joint Link3_Link4: type revolute, parent Link3, child Link4, origin xyz=0 1.0521541731407715 0 rpy=0 0 0, axis 1 0 0, limit lower=-3.14159 upper=3.14159 effort=0.0 velocity=0.0
- added joint Link4_Link5: type revolute, parent Link4, child Link5, origin xyz=0 0.8361161104843533 0 rpy=0 0 0, axis 1 0 0, limit lower=-3.14159 upper=3.14159 effort=0.0 velocity=0.0

Commit message: almost

File: body.urdf (robot description, URDF)
Before this commit: robot robot, 6 links, 5 joints
Links:
- removed link Link0
- removed link Link1
- removed link Link2
- removed link Link3
- removed link Link4
- removed link Link5
- added link 0, mass 1; collision box size=0.2654685243743693 1.2232740110121312 1.2261938877498246; visual box size=0.2654685243743693 1.2232740110121312 1.2261938877498246
- added link 1, mass 1; collision box size=0.2399499551929954 1.3890973649974612 0.27631980982003407; visual box size=0.2399499551929954 1.3890973649974612 0.27631980982003407
- added link 2, mass 1; collision box size=0.032596006916480846 0.10541950635963288 0.7892374078678929; visual box size=0.032596006916480846 0.10541950635963288 0.7892374078678929
- added link 3, mass 1; collision box size=0.07375234235388084 1.0390185617296817 0.04449790546995064; visual box size=0.07375234235388084 1.0390185617296817 0.04449790546995064
- added link 4, mass 1; collision box size=0.765405171750938 0.40520633816256596 0.008402180048944996; visual box size=0.765405171750938 0.40520633816256596 0.008402180048944996
- added link 5, mass 1; collision box size=0.3110586911523323 0.7809892207018478 0.24919585819318724; visual box size=0.3110586911523323 0.7809892207018478 0.24919585819318724
Joints:
- removed joint Link0_Link1
- removed joint Link1_Link2
- removed joint Link2_Link3
- removed joint Link3_Link4
- removed joint Link4_Link5
- added joint 0_1: type revolute, parent 0, child 1, origin xyz=0.05942037966875571 0.6116370055060656 0.43054596753843666 rpy=0 0 0, axis 0 0 1, limit lower=-3.14159 upper=3.14159 effort=0.0 velocity=0.0
- added joint 0_2: type revolute, parent 0, child 2, origin xyz=-0.09188572785495112 -0.41023665510001317 1.2261938877498246 rpy=0 0 0, axis 1 0 0, limit lower=-3.14159 upper=3.14159 effort=0.0 velocity=0.0
- added joint 0_3: type revolute, parent 0, child 3, origin xyz=0.0934854113866154 0.6116370055060656 1.0792568680939978 rpy=0 0 0, axis 0 0 1, limit lower=-3.14159 upper=3.14159 effort=0.0 velocity=0.0
- added joint 0_4: type revolute, parent 0, child 4, origin xyz=0.13273426218718465 0.026126045936202047 0.11291494438569903 rpy=0 0 0, axis 0 0 1, limit lower=-3.14159 upper=3.14159 effort=0.0 velocity=0.0
- added joint 0_5: type revolute, parent 0, child 5, origin xyz=-0.09419832386929954 0.6116370055060656 0.03758213091478424 rpy=0 0 0, axis 0 0 1, limit lower=-3.14159 upper=3.14159 effort=0.0 velocity=0.0
